File: ClassAA-amp/ClassAA-amp.kicad_sch (KiCad schematic)
At the start: 30 parts, among them J1 XH_3pin, J2 AudioJack3, J3 AudioJack3, U1 NJM4580DD, U2 NJM4556AD

Commit message: 電源に電解コンデンサ追加
470uF
Parts:
- added C10, C9: 470u, symbol Device:C_Polarized
Connections:
- net GND: now also C10.1, C9.2
- net VEE: now also C10.2
- net VDD renamed VCC
- net VCC: now also C9.1
Other:
- moved on the sheet: C1, C2, C3, C4, U1C, U2C
